Commit message: [tool-frame] added fixes from gaya

File: urdf/armar6.urdf (robot description, URDF)
Before this commit: robot Armar6, 59 links, 58 joints
Joints:
- joint left_tool_frame_joint: origin xyz=0.15 -0.1 0.01 rpy=1.57 0 0 -> xyz=0.15 -0.07 0.01 rpy=1.57 0 0.7854
- joint right_tool_frame_joint: origin xyz=0.15 -0.1 -0.01 rpy=1.57 0 0 -> xyz=0.15 -0.07 -0.01 rpy=1.57 0 0.7854
